Commit message: Gazeboモデルでの動作確認を完了

File: urdf/mecanum_wheel_macro.xacro (robot description, xacro)
@@ -3,7 +3,21 @@
   <xacro:include filename="$(find mecanum_wheel_description)/urdf/wheel.xacro" />
   <xacro:include filename="$(find mecanum_wheel_description)/urdf/rollers.xacro"  />
-  <xacro:macro name="mecanum_wheel" params="name side">
+  <xacro:macro name="mecanum_wheel" params="name side interface">
     <xacro:wheel_link name="${name}" side="${side}" />
     <xacro:rollers_link name="${name}" side="${side}" />
+    <transmission name="${name}_trans">
+      <type>transmission_interface/SimpleTransmission</type>
+      <joint name="${name}_joint">
+        <!-- <hardwareInterface>hardware_interface/EffortJointInterface</hardwareInterface> -->
+        <!-- <hardwareInterface>hardware_interface/VelocityJointInterface</hardwareInterface> -->
+        <hardwareInterface>${interface}</hardwareInterface>
+      </joint>
+      <actuator name="${name}_motor">
+        <!-- <hardwareInterface>hardware_interface/EffortJointInterface</hardwareInterface> -->
+        <!-- <hardwareInterface>hardware_interface/VelocityJointInterface</hardwareInterface> -->
+        <hardwareInterface>${interface}</hardwareInterface>
+        <mechanismReduction>1</mechanismReduction>
+      </actuator>
+    </transmission>
   </xacro:macro>
 </robot>

File: urdf/rollers.xacro (robot description, xacro)
@@ -25,8 +25,8 @@
         <inertial>
           <origin xyz="0 0 0" />
-          <mass value="1.0" />
-          <inertia ixx="1.0" ixy="0.0" ixz="0.0"
-                  iyy="1.0" iyz="0.0"
-                  izz="1.0" />
+          <mass value="0.3" />
+          <inertia ixx="0.00024000" ixy="0.0" ixz="0.0"
+                  iyy="0.00076000" iyz="0.0"
+                  izz="0.00076000" />
         </inertial>
       </link>
@@ -35,5 +35,13 @@
         <parent link="${name}_wheel_link" />
         <child link="${name}_roller${loop}_link" />
+        <dynamics damping="0.01" friction="0.0001" />
       </joint>
+      <gazebo reference="${name}_roller${loop}_link">
+        <mu1 value="0.6"/>
+        <mu2 value="0.6"/>
+        <kp value="10000000.0" />
+        <kd value="1.0" />
+        <fdir1 value="0 1 0"/>
+      </gazebo>
       <xacro:roller_loop name="${name}" side="${side}" num="${num}" loop="${loop - 1}" />
     </xacro:if>

File: urdf/wheel.xacro (robot description, xacro)
@@ -16,10 +16,17 @@
       <inertial>
         <origin xyz="0 0 0" />
-        <mass value="1.0" />
-        <inertia ixx="1.0" ixy="0.0" ixz="0.0"
-                iyy="1.0" iyz="0.0"
-                izz="1.0" />
+        <mass value="2.0" />
+        <inertia ixx="0.042025" ixy="0.0" ixz="0.0"
+                iyy="0.024279" iyz="0.0"
+                izz="0.024279" />
       </inertial>
     </link>
+    <gazebo reference="${name}_wheel_link">
+      <mu1 value="0.6"/>
+      <mu2 value="0.6"/>
+      <kp value="10000000.0" />
+      <kd value="1.0" />
+      <fdir1 value="0 1 0"/>
+    </gazebo>
   </xacro:macro>
 </robot>
