Commit message: ローラジョイント方向を修正

File: urdf/rollers.xacro (robot description, xacro)
@@ -1,5 +1,13 @@
 <?xml version="1.0" ?>
 <robot name="wheel" xmlns:xacro="http://www.ros.org/wiki/xacro">
-  <xacro:macro name="roller_loop" params="name num loop" >
+  <xacro:macro name="roller_origin" params="th side" >
+    <xacro:if value="${side==1}">
+      <origin xyz="0 ${0.0895*cos(th)} ${0.0895*sin(th)}" rpy="${atan(-tan(th)*sqrt(2.0))} ${asin(cos(th)/sqrt(2.0))} ${atan(sin(th))}"/>
+    </xacro:if>
+    <xacro:if value="${side==-1}">
+      <origin xyz="0 ${0.0895*cos(th)} ${0.0895*sin(th)}" rpy="${atan(-tan(th)*sqrt(2.0))} ${asin(-cos(th)/sqrt(2.0))} ${atan(-sin(th))}"/>
+    </xacro:if>
+  </xacro:macro>
+  <xacro:macro name="roller_loop" params="name side num loop" >
     <xacro:if value="${loop}">
       <link name="${name}_roller${loop}_link">
@@ -24,13 +32,13 @@
       </link>
       <joint name="${name}_roller${loop}_joint" type="fixed">
-        <origin xyz="0 ${0.0895*cos(radians(360/num*(loop-1)))} ${0.0895*sin(radians(360/num*(loop-1)))}" rpy="${radians(360/num*(loop-1))} ${radians(45)} 0 "/>
+        <xacro:roller_origin th="${radians(360/num*(loop-1))}" side="${side}"/>
         <parent link="${name}_wheel_link" />
         <child link="${name}_roller${loop}_link" />
       </joint>
-      <xacro:roller_loop name="${name}" num="${num}" loop="${loop - 1}" />
+      <xacro:roller_loop name="${name}" side="${side}" num="${num}" loop="${loop - 1}" />
     </xacro:if>
   </xacro:macro>
   <xacro:macro name="rollers_link" params="name side">
-    <xacro:roller_loop name="${name}" num="5" loop="5" />
+    <xacro:roller_loop name="${name}" side="${side}" num="15" loop="15" />
   </xacro:macro>
 </robot>

Commit message: ローラジョイントを無限回転ジョイントへ変更

File: urdf/rollers.xacro (robot description, xacro)
@@ -31,5 +31,5 @@
         </inertial>
       </link>
-      <joint name="${name}_roller${loop}_joint" type="fixed">
+      <joint name="${name}_roller${loop}_joint" type="continuous">
         <xacro:roller_origin th="${radians(360/num*(loop-1))}" side="${side}"/>
         <parent link="${name}_wheel_link" />

Commit message: gazebo joint state correspndence

File: urdf/rollers.xacro (robot description, xacro)
@@ -35,9 +35,19 @@
         <parent link="${name}_wheel_link" />
         <child link="${name}_roller${loop}_link" />
-        <dynamics damping="0.01" friction="0.0001" />
+        <dynamics damping="0.001" friction="0.0001" />
       </joint>
+      <transmission name="$${name}_roller${loop}_trans">
+        <type>transmission_interface/SimpleTransmission</type>
+        <joint name="${name}_roller${loop}_joint">
+          <hardwareInterface>hardware_interface/EffortJointInterface</hardwareInterface>
+        </joint>
+        <actuator name="${name}_roller${loop}_motor">
+          <hardwareInterface>hardware_interface/EffortJointInterface</hardwareInterface>
+          <mechanismReduction>1</mechanismReduction>
+        </actuator>
+      </transmission>
       <gazebo reference="${name}_roller${loop}_link">
-        <mu1 value="0.6"/>
-        <mu2 value="0.6"/>
+        <mu1 value="0.8"/>
+        <mu2 value="0.8"/>
         <kp value="10000000.0" />
         <kd value="1.0" />

Commit message: Jointに軸方向を追加

File: urdf/rollers.xacro (robot description, xacro)
@@ -33,4 +33,5 @@
       <joint name="${name}_roller${loop}_joint" type="continuous">
         <xacro:roller_origin th="${radians(360/num*(loop-1))}" side="${side}"/>
+        <axis xyz="1 0 0"/>
         <parent link="${name}_wheel_link" />
         <child link="${name}_roller${loop}_link" />
