Commit message: パッケージ名称を変更

File: test/test_robot.urdf.xacro (robot description, xacro)
@@ -1,5 +1,5 @@
 <?xml version="1.0" ?>
 <robot name="mecanum_wheel_robot" xmlns:xacro="http://ros.org/wiki/xacro">
-  <xacro:include filename="$(find mecanum_wheel_description)/urdf/mecanum_wheel_macro.xacro" />
+  <xacro:include filename="$(find fuji_mecanum)/urdf/mecanum_wheel_macro.xacro" />
   <link name="base_link">
     <visual>

File: urdf/mecanum_wheel.urdf.xacro (robot description, xacro)
@@ -1,7 +1,7 @@
 <?xml version="1.0" ?>
 <robot name="mecanum_wheel_robot" xmlns:xacro="http://ros.org/wiki/xacro">
-  <xacro:include filename="$(find mecanum_wheel_description)/urdf/mecanum_wheel_macro.xacro" />
-  <xacro:mecanum_wheel name="front_right" side="1" />
-  <xacro:mecanum_wheel name="front_left" side="-1" />
+  <xacro:include filename="$(find fuji_mecanum)/urdf/mecanum_wheel_macro.xacro" />
+  <xacro:mecanum_wheel name="front_right" side="1" interface="hardware_interface/EffortJointInterface" />
+  <xacro:mecanum_wheel name="front_left" side="-1" interface="hardware_interface/EffortJointInterface" />
   <link name="map">
     <origin xyz="0 0 0" rpy="0 0 0" />

File: urdf/mecanum_wheel_macro.xacro (robot description, xacro)
@@ -1,6 +1,6 @@
 <?xml version="1.0" ?>
 <robot name="mecanum_wheel" xmlns:xacro="http://ros.org/wiki/xacro">
-  <xacro:include filename="$(find mecanum_wheel_description)/urdf/wheel.xacro" />
-  <xacro:include filename="$(find mecanum_wheel_description)/urdf/rollers.xacro"  />
+  <xacro:include filename="$(find fuji_mecanum)/urdf/wheel.xacro" />
+  <xacro:include filename="$(find fuji_mecanum)/urdf/rollers.xacro"  />
   <xacro:macro name="mecanum_wheel" params="name side interface">
     <xacro:wheel_link name="${name}" side="${side}" />
@@ -9,11 +9,7 @@
       <type>transmission_interface/SimpleTransmission</type>
       <joint name="${name}_joint">
-        <!-- <hardwareInterface>hardware_interface/EffortJointInterface</hardwareInterface> -->
-        <!-- <hardwareInterface>hardware_interface/VelocityJointInterface</hardwareInterface> -->
         <hardwareInterface>${interface}</hardwareInterface>
       </joint>
       <actuator name="${name}_motor">
-        <!-- <hardwareInterface>hardware_interface/EffortJointInterface</hardwareInterface> -->
-        <!-- <hardwareInterface>hardware_interface/VelocityJointInterface</hardwareInterface> -->
         <hardwareInterface>${interface}</hardwareInterface>
         <mechanismReduction>1</mechanismReduction>

File: urdf/rollers.xacro (robot description, xacro)
@@ -15,10 +15,10 @@
           <origin xyz="0 0 0" rpy="0 0 0" />
           <geometry>
-            <mesh filename="package://mecanum_wheel_description/mesh/visual/roller.dae" scale="1 1 1" />
+            <mesh filename="package://fuji_mecanum/mesh/visual/roller.dae" scale="1 1 1" />
           </geometry>
         </visual>
         <collision>
           <geometry>
-            <mesh filename="package://mecanum_wheel_description/mesh/collision/roller.stl" scale="1 1 1" />
+            <mesh filename="package://fuji_mecanum/mesh/collision/roller.stl" scale="1 1 1" />
           </geometry>
         </collision>

File: urdf/wheel.xacro (robot description, xacro)
@@ -6,10 +6,10 @@
         <origin xyz="0 0 0" rpy="0 0 0" />
         <geometry>
-          <mesh filename="package://mecanum_wheel_description/mesh/visual/wheel.dae" scale="${side} 1 1" />
+          <mesh filename="package://fuji_mecanum/mesh/visual/wheel.dae" scale="${side} 1 1" />
         </geometry>
       </visual>
       <collision>
         <geometry>
-          <mesh filename="package://mecanum_wheel_description/mesh/collision/wheel.stl" scale="${side} 1 1" />
+          <mesh filename="package://fuji_mecanum/mesh/collision/wheel.stl" scale="${side} 1 1" />
         </geometry>
       </collision>

Commit message: ジョイント名称の変更

File: test/test_robot.urdf.xacro (robot description, xacro)
@@ -32,5 +32,5 @@
   <xacro:mecanum_wheel name="rear_right"  side="-1" interface="hardware_interface/EffortJointInterface"/>
   <xacro:mecanum_wheel name="rear_left"   side="1"  interface="hardware_interface/EffortJointInterface"/>
-  <joint name="front_right_joint" type="continuous">
+  <joint name="front_right_wheel_joint" type="continuous">
     <origin xyz="0.3 -0.25 -0.1" rpy="0 0 ${pi/2}" />
     <axis xyz="1 0 0" />
@@ -38,5 +38,5 @@
     <child link="front_right_wheel_link" />
   </joint>
-  <joint name="front_left_joint" type="continuous">
+  <joint name="front_left_wheel_joint" type="continuous">
     <origin xyz="0.3 0.25 -0.1" rpy="0 0 ${pi/2}" />
     <axis xyz="1 0 0" />
@@ -44,5 +44,5 @@
     <child link="front_left_wheel_link" />
   </joint>
-  <joint name="rear_right_joint" type="continuous">
+  <joint name="rear_right_wheel_joint" type="continuous">
     <origin xyz="-0.3 -0.25 -0.1" rpy="0 0 ${pi/2}" />
     <axis xyz="1 0 0" />
@@ -50,5 +50,5 @@
     <child link="rear_right_wheel_link" />
   </joint>
-  <joint name="rear_left_joint" type="continuous">
+  <joint name="rear_left_wheel_joint" type="continuous">
     <origin xyz="-0.3 0.25 -0.1" rpy="0 0 ${pi/2}" />
     <axis xyz="1 0 0" />

File: urdf/mecanum_wheel_macro.xacro (robot description, xacro)
@@ -6,10 +6,10 @@
     <xacro:wheel_link name="${name}" side="${side}" />
     <xacro:rollers_link name="${name}" side="${side}" />
-    <transmission name="${name}_trans">
+    <transmission name="${name}_wheel_trans">
       <type>transmission_interface/SimpleTransmission</type>
-      <joint name="${name}_joint">
+      <joint name="${name}_wheel_joint">
         <hardwareInterface>${interface}</hardwareInterface>
       </joint>
-      <actuator name="${name}_motor">
+      <actuator name="${name}_wheel_motor">
         <hardwareInterface>${interface}</hardwareInterface>
         <mechanismReduction>1</mechanismReduction>
